File: IC_circuit.kicad_sch (KiCad schematic)
At the start: 0 parts

Commit message: Added nRF54L10 circuitry
Parts:
- added C1: 1.5 pF, symbol Device:C
- added C10, C11, C8, C9: 100 nF, symbol Device:C
- added C2: 2.0 pF, symbol Device:C
- added C3: 0.3 pF, symbol Device:C
- added C4, C6: 2.2 uF, symbol Device:C
- added C5: 2.2 nF, symbol Device:C
- added C7: 10 nF, symbol Device:C
- added FB1: 120 ohm, symbol Device:FerriteBead_Small
- added IC1: NRF54L10-QFAA-R, QFN40P600X600X90-49N, symbol NRF54L10-QFAA-R:NRF54L10-QFAA-R
- added L1: 2.7 nH, symbol Device:L
- added L2, L3: 3.5 nH, symbol Device:L
- added L4: 4.7 uH, symbol Device:L
- added Y1: 32MHz, symbol Device:Crystal
Connections:
- new net: C2.1, L2.1, L3.2
- new net: C4.1, FB1.1, IC1.45 (DECD), L4.2
- new net: C1.1, L1.1, L2.2
- new net: IC1.31 (ANT), L1.2
- new net: IC1.34 (XC1), Y1.1
- new net: IC1.35 (XC2), Y1.2
- new net: IC1.46 (DCC), L4.1
- new net +3.3V: C10.1, C11.1, C8.1, C9.1, IC1.10 (VDD_1), IC1.22 (VDD_2), IC1.36 (VDD_3), IC1.47 (VDD_4), IC1.48 (VDD_5)
- new net Antenna: C3.1, L3.1
- new net Decoupling: C5.1, C6.1, C7.1, FB1.2, IC1.33 (DECRF), IC1.43 (DECA)
- new net GND: C1.2, C10.2, C11.2, C2.2, C3.2, C4.2, C5.2, C6.2, C7.2, C8.2, C9.2, IC1.32 (VSS_PA), IC1.44 (VSS), IC1.49 (EP)
Other:
- note added: "Note: C1 should be connected directly to pin 32"
- note added: "Note: C2 should be connected only to the bottom layer GND pour"
- note added: "Note: Pin 32 should be connected directly to the die pad (pin 49)"
- note added: "uC nRF54L10"
