File: Power_circuit.kicad_sch (KiCad schematic)
At the start: 0 parts

Commit message: Eighth commit, basic power circuit, need to select values and run simulations
Parts:
- added C1: C, symbol Device:C
- added C2, C3: C_US, symbol Device:C_US
- added D1: MB2S, symbol Custom_Symbols:MB2S
- added D2, D3: 1N914, Diode_THT:D_DO-35_SOD27_P7.62mm_Horizontal, symbol Diode:1N914
- added J1: (no value), symbol Custom_Symbols:Power_Prongs
- added L1: L, symbol Device:L
- added R1, R2, R3, R4: R, symbol Device:R
- added U1: LNK3206D, Package_SO:PowerIntegrations_SO-8C, symbol Regulator_Switching:LNK3206D
Connections:
- new net: C1.2, C2.2, D3.1 (K), L1.1, R1.2, U1.5 (S), U1.6 (S), U1.7 (S), U1.8 (S)
- new net: C2.1, D2.1 (K), R2.2, R3.2
- new net: C1.1, R3.1, U1.1 (BP/M)
- new net: D1.4, J1. (N)
- new net: D1.3, J1.1 (H)
- new net: R1.1, R2.1, U1.2 (FB)
- new net: D1.1 (+), U1.4 (D)
- new net GND: C3.2, D1.2 (-), D3.2 (A), R4.2
- new net VDC: C3.1, D2.2 (A), L1.2, R4.1
